Commit message: RPLidar tests

File: create_description/urdf/create_base.urdf.xacro (robot description, xacro)
@@ -197,8 +197,45 @@
     </inertial>
     </link>
+  <xacro:macro name="cylinder_inertia" params="mass r l">
+    <!-- <inertia
+      ixx="${mass*(3*r*r + l*l)/12}" ixy="0" ixz="0"
+      iyy="${mass*(3*r*r + l*l)/12}" iyz="0"
+      izz="${mass*(r*r)/2}" /> -->
+    <inertia
+      ixx="0" ixy="0" ixz="0"
+      iyy="0" iyz="0"
+      izz="0" />
+  </xacro:macro>
     <!-- Simulation sensors -->
     <xacro:sim_create_base/>
     <xacro:sim_create_wall_sensor/>
     <xacro:sim_create_cliff_sensors/>
+    <link name="laser">
+      <inertial>
+        <origin xyz="0 0 0" rpy="0 0 0" />
+        <mass value="1" />
+        <xacro:cylinder_inertia mass="1.0" r="${radius}" l="{height}" />
+      </inertial>
+      <visual>
+        <origin xyz="0 0 0" rpy="0 0 0" />
+        <geometry>
+          <cylinder radius="${radius}" length="${height}"/>
+        </geometry>
+        <material name="White">
+          <color rgba="0.85 0.85 0.85 1.0" />
+        </material>
+      </visual>
+        <collision>
+          <origin xyz="0.0 0.0 0.0" rpy="0.0 0.0 0.0"/>
+          <geometry>
+            <cylinder radius="${radius}" length="${height}"/>
+          </geometry>
+        </collision>
+    </link>
+    <joint name="joint_sensor_laser" type="fixed">
+      <origin xyz="${x_offset} ${y_offset} ${z_offset}" rpy="0.0 0.0 0.0"/>
+      <parent link="base_link"/>
+      <child link="laser"/>
+    </joint>
     <xacro:sim_imu/>
   </xacro:macro>

Commit message: Fix robot model

File: create_description/urdf/create_base.urdf.xacro (robot description, xacro)
@@ -207,8 +207,5 @@
       izz="0" />
   </xacro:macro>
-    <!-- Simulation sensors -->
-    <xacro:sim_create_base/>
-    <xacro:sim_create_wall_sensor/>
-    <xacro:sim_create_cliff_sensors/>
+  <xacro:macro name="create_laser" params="x_offset y_offset z_offset height radius">
     <link name="laser">
       <inertial>
@@ -223,13 +220,13 @@
         </geometry>
         <material name="White">
-          <color rgba="0.85 0.85 0.85 1.0" />
+           <color rgba="0.85 0.85 0.85 1.0" />
         </material>
       </visual>
-        <collision>
-          <origin xyz="0.0 0.0 0.0" rpy="0.0 0.0 0.0"/>
-          <geometry>
-            <cylinder radius="${radius}" length="${height}"/>
-          </geometry>
-        </collision>
+      <collision>
+        <origin xyz="0.0 0.0 0.0" rpy="0.0 0.0 0.0"/>
+        <geometry>
+          <cylinder radius="${radius}" length="${height}"/>
+        </geometry>
+      </collision>
     </link>
     <joint name="joint_sensor_laser" type="fixed">
@@ -238,4 +235,10 @@
       <child link="laser"/>
     </joint>
+  </xacro:macro>
+    <!-- Simulation sensors -->
+    <xacro:sim_create_base/>
+    <xacro:sim_create_wall_sensor/>
+    <xacro:sim_create_cliff_sensors/>
+    <xacro:create_laser x_offset="-0.03" y_offset="-0.01" z_offset="0.180" radius="0.035" height="0.025" />
     <xacro:sim_imu/>
   </xacro:macro>
